File: ebike-charger.kicad_sch (KiCad schematic)
At the start: 0 parts

Commit message: syncing
Other:
- sheet Ideal Diode (Anti-Backfeed) renamed Ideal Diode (Anti-Backfeed) and Output
- removed sheet Output
- sheet Boost Converter ports: added V_CHARGE; removed none
- sheet Ideal Diode (Anti-Backfeed) and Output: file ideal-diode.kicad_sch -> ideal-diode-output.kicad_sch
Changed lines of the file:
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@@
-	)
-	(sheet
-		(at 241.3 63.5)
-		(size 25.4 38.1)
-		(exclude_from_sim no)
-		(in_bom yes)
-		(on_board yes)
-		(dnp no)
-		(fields_autoplaced yes)
-		(stroke
-			(width 0.1524)
-			(type solid)
-		)
-		(fill
-			(color 0 0 0 0)
-		)
-		(property "Sheetname" "Output"
-			(at 241.3 62.7884 0)
-			(show_name no)
-			(do_not_autoplace no)
-			(effects
-				(font
-					(size 1.27 1.27)
-				)
-				(justify left bottom)
-			)
-		)
-		(property "Sheetfile" "output.kicad_sch"
-			(at 241.3 102.1846 0)
-			(show_name no)
-			(do_not_autoplace no)
-			(effects
-				(font
-					(size 1.27 1.27)
-				)
-				(justify left top)
-			)
-		)
-		(instances
-			(project "ebike-charger"
-				(path "/9487e442-8735-4068-9b97-626a2310d20e"
-					(page "6")
-				)
-			)
-		)
 	)
 	(sheet
@@
 			(color 0 0 0 0)
 		)
-		(property "Sheetname" "Ideal Diode (Anti-Backfeed)"
+		(property "Sheetname" "Ideal Diode (Anti-Backfeed) and Output"
 			(at 190.5 62.7884 0)
 			(show_name no)
@@
 			)
 		)
-		(property "Sheetfile" "ideal-diode.kicad_sch"
+		(property "Sheetfile" "ideal-diode-output.kicad_sch"
 			(at 190.5 102.1846 0)
 			(show_name no)
@@
 			)
 		)
+		(pin "V_CHARGE" input
+			(at 114.3 67.31 0)
+			(effects
+				(font
+					(size 1.27 1.27)
+				)
+				(justify right)
+			)
+		)
