File: boost-converter.kicad_sch (KiCad schematic)
At the start: 23 parts, among them Q1 CSD18543Q3A, Q2 CSD18543Q3A, U2 TPS43060RTER

Commit message: added ideal diode
Parts:
- renumbered Ccomp1 to Ccomp2
